Commit message: add files

File: dualarm_exhibition/urdf/dualarm_prbt.urdf.xacro (robot description, xacro)
@@ -78,6 +78,6 @@
   <joint name="table_joint" type="fixed">
 	<!-- <origin xyz="0 0 0" rpy="0 0 0" /> -->
-          <parent link="table" />
-          <child link="stander" />
+    <parent link="table" />
+    <child link="stander" />
   </joint>
   <link name="stander">
@@ -92,5 +92,5 @@
     </visual>
     <collision>
-      <origin xyz="0 0 0.2" rpy="0 0 0" />
+      <origin xyz="0 0.133 0.2" rpy="0 0 0" />
       <geometry>
         <cylinder radius="0.15" length="0.4" />
@@ -98,21 +98,21 @@
     </collision>
     <collision>
-      <origin xyz="0 0 0.41" rpy="0 0 0" />
+      <origin xyz="0 0.133 0.41" rpy="0 0 0" />
       <geometry>
         <sphere radius="0.21"/>
       </geometry>
     </collision>
-    <collision>
+    <!-- <collision>
       <origin xyz="0.05 0.13 0.43" rpy="0 0 0" />
       <geometry>
         <sphere radius="0.1"/>
       </geometry>
-    </collision>
-    <collision>
+    </collision> -->
+    <!-- <collision>
       <origin xyz="0.05 -0.13 0.43" rpy="0 0 0" />
       <geometry>
         <sphere radius="0.1"/>
       </geometry>
-    </collision>
+    </collision> -->
   </link>
   <!-- additional links for offset and rotation -->
